File: GitTest.kicad_sch (KiCad schematic)
At the start: 3 parts

Commit message: Route new SMD
Parts:
- D1: footprint LED_THT:LED_D3.0mm -> LED_SMD:LED_0603_1608Metric
- R1: footprint Resistor_THT:R_Axial_DIN0204_L3.6mm_D1.6mm_P5.08mm_Horizontal -> Resistor_SMD:R_0603_1608Metric
Changed lines of the file:
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@@
 			)
 		)
-		(property "Footprint" "LED_THT:LED_D3.0mm"
+		(property "Footprint" "LED_SMD:LED_0603_1608Metric"
 			(at 76.2 135.89 0)
 			(hide yes)
@@
 			)
 		)
-		(property "Footprint" "Resistor_THT:R_Axial_DIN0204_L3.6mm_D1.6mm_P5.08mm_Horizontal"
+		(property "Footprint" "Resistor_SMD:R_0603_1608Metric"
 			(at 74.422 123.19 90)
 			(hide yes)
